File: KiCAD/Howland-VCCS/Howland-VCCS-TL072_SMD/Howland-VCCS-TL072_SMD/Howland-VCCS-TL072_SMD.kicad_pcb (KiCad board)
At the start: 2 copper layers, 16 parts, among them J1 Conn_01x03_Pin, J2 Conn_01x03_Pin, U1 TL072

Commit message: Add Project Folder: KICAD
Parts:
- JP1, JP2: footprint Connector_PinHeader_2.54mm:PinHeader_1x03_P2.54mm_Vertical -> Jumper:SolderJumper-2_P1.3mm_Open_RoundedPad1.0x1.5mm

Commit message: Add Project Folder: KICAD
Parts:
- moved R6 36.6 mm to (189.1, 99.5), turned to 180 degrees
- moved R1 36.4 mm to (183.8, 99.5), turned to 180 degrees
- moved R2 33.0 mm to (183.8, 94.8)
- moved JP2 22.0 mm to (188.9, 95.0), turned to 180 degrees
- moved JP1 18.5 mm to (183.7, 89.2), turned to 180 degrees
- moved H1 16.8 mm to (141.5, 91.3)
- moved H2 16.8 mm to (141.5, 97.2)
- moved C1 12.6 mm to (160.0, 90.5)
- moved U1 11.4 mm to (170.2, 99.7)
- moved J2 6.92 mm to (167.9, 85.5), turned to 90 degrees
- moved J1 4.25 mm to (159.2, 85.5), turned to 90 degrees

Commit message: Add Project Folder: KICAD
Parts:
- C1, C2: footprint Capacitor_SMD:C_1206_3216Metric_Pad1.33x1.80mm_HandSolder -> Capacitor_SMD:C_0805_2012Metric
- H1, H2: footprint MountingHole:MountingHole_2.2mm_M2_Pad -> MountingHole:MountingHole_2.2mm_M2
- J1, J2: moved to B.Cu
- R1, R2, R3, R4, R5, R6, R7: footprint Resistor_SMD:R_1206_3216Metric -> Resistor_SMD:R_0805_2012Metric
- moved H2 58.6 mm to (199.7, 103.6)
- moved R5 43.6 mm to (196.1, 95.4), turned to 90 degrees
- moved H1 40.9 mm to (180.5, 103.6)
- moved C1 39.4 mm to (198.6, 98.4), turned to 90 degrees
- moved J1 36.8 mm to (195.9, 83.2)
- moved R7 33.3 mm to (183.6, 88.8)
- moved C2 32.2 mm to (191.8, 88.9), turned to 180 degrees
- moved R4 29.0 mm to (180.5, 98.4), turned to 90 degrees
- moved R3 28.4 mm to (180.5, 92.7), turned to -90 degrees
- moved J2 14.4 mm to (182.2, 83.2), turned to -90 degrees
- moved U1 13.8 mm to (184.0, 99.1), turned to 90 degrees
- moved R6 11.7 mm to (198.6, 92.7), turned to -90 degrees
- moved JP2 8.33 mm to (195.1, 100.6), turned to 90 degrees
- moved R2 7.95 mm to (185.6, 102.5), turned to 180 degrees
- moved R1 6.86 mm to (190.0, 102.5)
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Routing:
- net VEE: track 0.00 -> 22.6 mm
- net Net-(R2-Pad2): track 0.00 -> 18.9 mm, vias 0 -> 2
- net /Id+: track 0.00 -> 18.6 mm
- net Net-(C1-Pad2): track 0.00 -> 15.1 mm
- net /Out: track 0.00 -> 14.3 mm
- net Net-(U1A--): track 0.00 -> 13.9 mm
- net Net-(JP1-B): track 0.00 -> 12.8 mm
- net Net-(U1B--): track 0.00 -> 11.1 mm
- net VCC: track 0.00 -> 9.04 mm
- net Net-(U1A-+): track 0.00 -> 6.05 mm
- net /Id-: track 0.00 -> 6.00 mm
- net GND: vias 0 -> 3
- added copper zone on B.Cu, net GND
- added copper zone on F.Cu, net GND
Other:
- board outline added: 24.5 x 25.4 mm

Commit message: Add Project Folder: KICAD
Parts:
- moved R1 0.63 mm to (190.0, 103.1)
- moved R2 0.63 mm to (185.6, 103.1)
Routing:
- net Net-(R2-Pad2): track 18.9 -> 21.5 mm
- net Net-(U1A-+): track 6.05 -> 6.94 mm
- net Net-(C1-Pad2): track 15.1 -> 15.7 mm
- net GND: vias 3 -> 8
Changed lines of the file:
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@@
 	(footprint "Resistor_SMD:R_0805_2012Metric"
 		(layer "F.Cu")
-		(at 185.5705 102.497 180)
+		(at 185.5705 103.124 180)
 		(descr "Resistor SMD 0805 (2012 Metric), square (rectangular) end terminal, IPC-7351 nominal, (Body size source: IPC-SM-782 page 72, https://www.pcb-3d.com/wordpress/wp-content/uploads/ipc-sm-782a_amendment_1_and_2.pdf)")
 		(tags "resistor")
@@
 	(footprint "Resistor_SMD:R_0805_2012Metric"
 		(layer "F.Cu")
-		(at 189.992 102.497 180)
+		(at 189.992 103.124 180)
 		(descr "Resistor SMD 0805 (2012 Metric), square (rectangular) end terminal, IPC-7351 nominal, (Body size source: IPC-SM-782 page 72, https://www.pcb-3d.com/wordpress/wp-content/uploads/ipc-sm-782a_amendment_1_and_2.pdf)")
 		(tags "resistor")
@@
 	)
 	(segment
-		(start 190.9045 102.497)
-		(end 195.953 102.497)
+		(start 196.85 99.228)
+		(end 198.628 97.45)
 		(width 0.3)
 		(layer "F.Cu")
@@
 	)
 	(segment
-		(start 195.953 102.497)
-		(end 196.85 101.6)
+		(start 195.961 103.124)
+		(end 196.85 102.235)
 		(width 0.3)
 		(layer "F.Cu")
@@
 	)
 	(segment
-		(start 196.85 101.6)
+		(start 196.85 102.235)
 		(end 196.85 99.228)
 		(width 0.3)
@@
 	)
 	(segment
-		(start 196.85 99.228)
-		(end 198.628 97.45)
+		(start 190.9045 103.124)
+		(end 195.961 103.124)
 		(width 0.3)
 		(layer "F.Cu")
@@
 	)
 	(via
+		(at 185.8144 100.7364)
+		(size 0.6)
+		(drill 0.3)
+		(layers "F.Cu" "B.Cu")
+		(free yes)
+		(net "GND")
+	)
+	(via
+		(at 186.5256 100.7364)
+		(size 0.6)
+		(drill 0.3)
+		(layers "F.Cu" "B.Cu")
+		(free yes)
+		(net "GND")
+	)
+	(via
 		(at 189.357 89.408)
+		(size 0.6)
+		(drill 0.3)
+		(layers "F.Cu" "B.Cu")
+		(free yes)
+		(net "GND")
+	)
+	(via
+		(at 185.0644 100.7364)
+		(size 0.6)
+		(drill 0.3)
+		(layers "F.Cu" "B.Cu")
+		(free yes)
+		(net "GND")
+	)
+	(via
+		(at 187.8972 100.7364)
+		(size 0.6)
+		(drill 0.3)
+		(layers "F.Cu" "B.Cu")
+		(free yes)
+		(net "GND")
+	)
+	(via
+		(at 187.186 100.7364)
 		(size 0.6)
 		(drill 0.3)
@@
 	)
 	(segment
-		(start 189.0795 102.497)
-		(end 189.0795 102.2585)
+		(start 189.0795 103.124)
+		(end 189.0795 102.8855)
 		(width 0.2)
 		(layer "F.Cu")
@@
 	)
 	(segment
-		(start 189.0795 102.2585)
-		(end 189.1001 102.2379)
+		(start 189.0795 102.8855)
+		(end 189.1001 102.8649)
 		(width 0.2)
 		(layer "F.Cu")
@@
 	)
 	(segment
-		(start 189.1001 102.2379)
+		(start 189.1001 103.1034)
 		(end 189.1001 99.055)
 		(width 0.3)
@@
 	)
 	(segment
-		(start 189.0795 102.497)
-		(end 186.483 102.497)
+		(start 189.0795 103.124)
+		(end 186.483 103.124)
 		(width 0.3)
 		(layer "F.Cu")
@@
 	)
 	(segment
-		(start 187.96 100.33)
-		(end 185.2951 100.33)
+		(start 189.0795 103.124)
+		(end 189.1001 103.1034)
 		(width 0.3)
 		(layer "F.Cu")
+		(net "Net-(U1A-+)")
+	)
+	(segment
+		(start 184.9755 101.6)
+		(end 184.0201 100.6446)
+		(width 0.3)
+		(layer "F.Cu")
 		(net "Net-(R2-Pad2)")
 	)
 	(segment
-		(start 184.0201 101.8591)
-		(end 184.658 102.497)
+		(start 187.706 101.6)
+		(end 184.9755 101.6)
+		(width 0.3)
+		(layer "F.Cu")
+		(net "Net-(R2-Pad2)")
+	)
+	(segment
+		(start 184.0201 99.055)
+		(end 184.0201 102.4861)
+		(width 0.3)
+		(layer "F.Cu")
+		(net "Net-(R2-Pad2)")
+	)
+	(segment
+		(start 184.0201 100.6446)
+		(end 184.0201 99.055)
+		(width 0.3)
+		(layer "F.Cu")
+		(net "Net-(R2-Pad2)")
+	)
+	(segment
+		(start 184.0201 102.4861)
+		(end 184.658 103.124)
 		(width 0.3)
 		(layer "F.Cu")
@@
 		(end 194.7865 96.2975)
 		(width 0.2)
-		(layer "F.Cu")
-		(net "Net-(R2-Pad2)")
-	)
-	(segment
-		(start 185.2951 100.33)
-		(end 184.0201 99.055)
-		(width 0.3)
-		(layer "F.Cu")
-		(net "Net-(R2-Pad2)")
-	)
-	(segment
-		(start 184.0201 99.055)
-		(end 184.0201 101.8591)
-		(width 0.3)
 		(layer "F.Cu")
 		(net "Net-(R2-Pad2)")
@@
 	)
 	(via
-		(at 187.96 100.33)
+		(at 187.706 101.6)
 		(size 0.6)
 		(drill 0.3)
 		(layers "F.Cu" "B.Cu")
-		(net "Net-(R2-Pad2)")
-	)
-	(segment
-		(start 187.96 100.33)
-		(end 192.278 100.33)
-		(width 0.3)
-		(layer "B.Cu")
-		(net "Net-(R2-Pad2)")
-	)
-	(segment
-		(start 192.278 100.33)
-		(end 194.564 98.044)
-		(width 0.3)
-		(layer "B.Cu")
 		(net "Net-(R2-Pad2)")
 	)
@@
 		(layer "B.Cu")
 		(net "Net-(R2-Pad2)")
+	)
+	(segment
+		(start 187.706 101.6)
+		(end 191.008 101.6)
+		(width 0.3)
+		(layer "B.Cu")
+		(net "Net-(R2-Pad2)")
+	)
+	(segment
+		(start 191.008 101.6)
+		(end 194.564 98.044)
+		(width 0.3)
+		(layer "B.Cu")
+		(net "Net-(R2-Pad2)")
