File: KiCAD/Howland-VCCS/Howland-VCCS-TL072_SMD - Copy/Howland-VCCS-TL072_SMD_2/Howland-VCCS-TL072_SMD_2.kicad_pcb (KiCad board)
At the start: 2 copper layers, 24.5 x 25.4 mm, 16 parts, among them J1 Conn_01x03_Pin, J2 Conn_01x03_Pin, U1 TL072

Commit message: Add Project Folder: KICAD
Parts:
- moved J2 24.2 mm to (192.4, 105.1), turned to 90 degrees
- moved C1 21.5 mm to (180.2, 87.4), turned to -90 degrees
- moved R3 16.6 mm to (196.2, 87.4), turned to 180 degrees
- moved R1 16.4 mm to (183.6, 87.4), turned to 0 degrees
- moved R4 15.9 mm to (196.2, 100.8), turned to 180 degrees
- moved R6 15.9 mm to (182.8, 91.1), turned to 90 degrees
- moved R2 15.3 mm to (187.9, 87.4), turned to 0 degrees
- moved R7 13.7 mm to (197.1, 91.1), turned to -90 degrees
- moved U1 13.4 mm to (193.8, 89.9), turned to -90 degrees
- moved JP2 12.9 mm to (182.8, 96.7)
- moved JP1 12.8 mm to (197.1, 96.7)
- moved H1 9.88 mm to (178.4, 94.0)
- moved H2 9.82 mm to (201.6, 93.9)
- moved R5 8.97 mm to (192.0, 87.4), turned to 0 degrees
- moved J1 8.56 mm to (187.4, 83.3), turned to -90 degrees
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Routing:
- net VEE: track 22.6 -> 0.00 mm
- net Net-(R2-Pad2): track 18.9 -> 0.00 mm, vias 2 -> 0
- net /Id+: track 18.6 -> 0.00 mm
- net Net-(C1-Pad2): track 15.1 -> 0.00 mm
- net /Out: track 14.3 -> 0.00 mm
- net Net-(U1A--): track 13.9 -> 0.00 mm
- net Net-(JP1-B): track 12.8 -> 0.00 mm
- net Net-(U1B--): track 11.1 -> 0.00 mm
- net VCC: track 9.04 -> 0.00 mm
- net Net-(U1A-+): track 6.05 -> 0.00 mm
- net /Id-: track 6.00 -> 0.00 mm
- net GND: vias 3 -> 0
Other:
- board size 24.5 x 25.4 mm -> 29.4 x 27.3 mm

Commit message: Add Project Folder: KICAD
Parts:
- moved R3 6.57 mm to (197.5, 93.8), turned to -90 degrees
- moved R4 6.22 mm to (190.0, 100.9)
- moved JP2 3.65 mm to (182.7, 100.4)
- moved JP1 3.57 mm to (197.5, 100.3)
- moved R1 2.77 mm to (186.3, 87.4)
- moved R6 2.72 mm to (182.7, 93.9)
- moved C1 2.54 mm to (182.7, 87.4)
- moved R2 2.14 mm to (190.0, 87.4)
- moved C2 2.08 mm to (197.5, 87.4)
- moved R5 1.58 mm to (193.6, 87.4)
- moved R7 0.58 mm to (197.5, 90.6), turned to 180 degrees
Routing:
- net /Out: track 0.00 -> 32.7 mm
- net VEE: track 0.00 -> 20.7 mm
- net Net-(U1A--): track 0.00 -> 16.7 mm
- net Net-(JP1-B): track 0.00 -> 12.9 mm
- net /Id-: track 0.00 -> 12.1 mm
- net VCC: track 0.00 -> 8.12 mm
- net Net-(C1-Pad2): track 0.00 -> 7.71 mm
- net Net-(U1B--): track 0.00 -> 6.03 mm
- net /Id+: track 0.00 -> 5.90 mm
- net Net-(R2-Pad2): track 0.00 -> 4.81 mm
- net Net-(U1A-+): track 0.00 -> 4.54 mm
