File: KiCAD/Howland-VCCS/Howland-VCCS-TL072/Howland-VCCS-TL072.kicad_pcb (KiCad board)
At the start: 2 copper layers, 16 parts, among them J1 Conn_01x03_Pin, J2 Conn_01x03_Pin, U1 TL072

Commit message: Add Project Folder: KICAD
Parts:
- JP1, JP2: footprint Connector_PinHeader_2.54mm:PinHeader_1x03_P2.54mm_Vertical -> Jumper:SolderJumper-2_P1.3mm_Open_RoundedPad1.0x1.5mm
- moved R7 69.5 mm to (213.4, 86.4), turned to 90 degrees
- moved R4 64.3 mm to (208.3, 76.2), turned to -90 degrees
- moved R3 60.1 mm to (203.2, 86.4), turned to 90 degrees
- moved R5 58.0 mm to (200.7, 71.1)
- moved C2 57.5 mm to (213.9, 71.1)
- moved H2 55.9 mm to (221.0, 78.7)
- moved J2 44.7 mm to (200.7, 91.4), turned to -90 degrees
- moved R2 41.6 mm to (185.4, 76.2), turned to -90 degrees
- moved R1 41.5 mm to (185.4, 71.1)
- moved J1 37.5 mm to (195.6, 66.0), turned to 90 degrees
- moved U1 36.5 mm to (198.1, 76.2), turned to -90 degrees
- moved R6 36.3 mm to (180.3, 86.4), turned to 90 degrees
- moved JP1 33.8 mm to (188.6, 94.0)
- moved JP2 26.9 mm to (188.6, 88.9)
- moved C1 21.5 mm to (178.3, 71.1)
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Routing:
- net Net-(JP1-B): track 0.00 -> 55.9 mm
- net GND: track 0.00 -> 51.2 mm
- net Net-(R2-Pad2): track 0.00 -> 42.3 mm
- net /Out: track 0.00 -> 40.8 mm
- net Net-(U1B--): track 0.00 -> 24.3 mm
- net VEE: track 0.00 -> 23.1 mm
- net /Id+: track 0.00 -> 19.3 mm, vias 0 -> 1
- net /Id-: track 0.00 -> 18.8 mm
- net Net-(U1A-+): track 0.00 -> 14.7 mm
- net Net-(U1A--): track 0.00 -> 13.6 mm
- net Net-(C1-Pad2): track 0.00 -> 10.2 mm
- net VCC: track 0.00 -> 8.67 mm
- net (no net): vias 0 -> 92
Other:
- board outline added: 50.8 x 33 mm

Commit message: Add Project Folder: KICAD
Routing:
- net /Id+: vias 1 -> 0
- net (no net): vias 92 -> 209
Other:
- board size 50.8 x 33 mm -> 61.1 x 40.1 mm

Commit message: Add Project Folder: KICAD
Parts:
- removed C1, C2: C, Capacitor_THT:C_Radial_D5.0mm_H11.0mm_P2.00mm
- removed H1, H2: MountingHole, MountingHole:MountingHole_2.2mm_M2_Pad
- removed JP1, JP2: SolderJumper_2_Open, Jumper:SolderJumper-2_P1.3mm_Open_RoundedPad1.0x1.5mm
Connections:
- J1 pad 2: /Id- -> GND
- R1 pad 1: Net-(C1-Pad2) -> /Id+
- R3 pad 1: Net-(JP1-B) -> GND
Routing:
- net Net-(JP1-B): track 55.9 -> 0.00 mm
- net GND: track 51.2 -> 107.0 mm
- net /Out: track 40.8 -> 94.3 mm
- net /Id-: track 18.8 -> 0.00 mm
- net Net-(R2-Pad2): track 42.3 -> 33.6 mm
- net Net-(U1B--): track 24.3 -> 18.4 mm
- net /Id+: track 19.3 -> 13.8 mm
- net VEE: track 23.1 -> 26.5 mm
- net Net-(U1A--): track 13.6 -> 14.8 mm
- net Net-(U1A-+): track 14.7 -> 15.9 mm
- net (no net): vias 209 -> 12

Commit message: Add Project Folder: KICAD
Parts:
- removed R6, R7: R, Resistor_THT:R_Axial_DIN0207_L6.3mm_D2.5mm_P10.16mm_Horizontal
- added RV1: 1K, Potentiometer_THT:Potentiometer_Bourns_3296W_Vertical, F.Cu at (215.9, 88.9)
- R2, R4: value 20k -> 100k
- R5: value 100 -> 150
Routing:
- net Net-(R2-Pad2): track 33.6 -> 76.8 mm
- net GND: track 107.0 -> 77.4 mm
- net Net-(C1-Pad2): track 10.2 -> 0.00 mm
- net /Out: track 94.3 -> 88.6 mm
- net (no net): vias 12 -> 180
