File: KiCAD/Howland-VCCS/Howland-VCCS-TL072/Howland-VCCS-TL072.kicad_sch (KiCad schematic)
At the start: 0 parts

Commit message: Add Project Folder: KICAD
Parts:
- added C1, C2: C, Capacitor_THT:C_Radial_D5.0mm_H11.0mm_P2.00mm, symbol Device:C
- added H1, H2: MountingHole, MountingHole:MountingHole_2.2mm_M2_Pad, symbol Mechanical:MountingHole
- added J1, J2: Conn_01x03_Pin, Connector_PinHeader_2.54mm:PinHeader_1x03_P2.54mm_Vertical, symbol Connector:Conn_01x03_Pin
- added JP1, JP2: SolderJumper_2_Open, Connector_PinHeader_2.54mm:PinHeader_1x03_P2.54mm_Vertical, symbol Jumper:SolderJumper_2_Open
- added R1, R3: 100k, Resistor_THT:R_Axial_DIN0207_L6.3mm_D2.5mm_P10.16mm_Horizontal, symbol Device:R
- added R2, R4: 20k, Resistor_THT:R_Axial_DIN0207_L6.3mm_D2.5mm_P10.16mm_Horizontal, symbol Device:R
- added R5: 100, Resistor_THT:R_Axial_DIN0207_L6.3mm_D2.5mm_P10.16mm_Horizontal, symbol Device:R
- added R6, R7: R, Resistor_THT:R_Axial_DIN0207_L6.3mm_D2.5mm_P10.16mm_Horizontal, symbol Device:R
- added U1: TL072, Package_DIP:DIP-8_W7.62mm, symbol Amplifier_Operational:TL072
Connections:
- new net: R1.2, R2.1, U1.3 (+)
- new net: R2.2, R5.1, U1.1
- new net: C2.2, JP1.2 (B), R3.1, R7.2
- new net: C1.2, R1.1, R6.2
- new net: R4.2, U1.6 (-), U1.7
- new net: R3.2, R4.1, U1.2 (-)
- new net GND: J2.3 (Pin_3), JP1.1 (A), JP2.1 (A), R6.1, R7.1
- new net Id+: C1.1, J1.1 (Pin_1)
- new net Id-: C2.1, J1.2 (Pin_2)
- new net Out: J1.3 (Pin_3), R5.2, U1.5 (+)
- new net VCC: J2.1 (Pin_1), U1.8 (V+)
- new net VEE: J2.2 (Pin_2), JP2.2 (B), U1.4 (V-)
Other:
- note added: "Current Out"
- note added: "In INV"
- note added: "In Non-INV"
- note added: "PWR+"
- note added: "PWR-"

Commit message: Add Project Folder: KICAD
Parts:
- JP1, JP2: footprint Connector_PinHeader_2.54mm:PinHeader_1x03_P2.54mm_Vertical -> Jumper:SolderJumper-2_P1.3mm_Open_RoundedPad1.0x1.5mm
Changed lines of the file:
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@@
 			)
 		)
-		(property "Footprint" "Connector_PinHeader_2.54mm:PinHeader_1x03_P2.54mm_Vertical"
+		(property "Footprint" "Jumper:SolderJumper-2_P1.3mm_Open_RoundedPad1.0x1.5mm"
 			(at 76.2 102.87 0)
 			(hide yes)
@@
 			)
 		)
-		(property "Footprint" "Connector_PinHeader_2.54mm:PinHeader_1x03_P2.54mm_Vertical"
+		(property "Footprint" "Jumper:SolderJumper-2_P1.3mm_Open_RoundedPad1.0x1.5mm"
 			(at 144.78 116.84 0)
 			(hide yes)

Commit message: Add Project Folder: KICAD
Parts:
- removed C1, C2: C, Capacitor_THT:C_Radial_D5.0mm_H11.0mm_P2.00mm, symbol Device:C
- removed H1, H2: MountingHole, MountingHole:MountingHole_2.2mm_M2_Pad, symbol Mechanical:MountingHole
- removed JP1, JP2: SolderJumper_2_Open, Jumper:SolderJumper-2_P1.3mm_Open_RoundedPad1.0x1.5mm, symbol Jumper:SolderJumper_2_Open
- removed R6, R7: R, Resistor_THT:R_Axial_DIN0207_L6.3mm_D2.5mm_P10.16mm_Horizontal, symbol Device:R
Connections:
- net Id- is gone; now on net GND: J1.2 (Pin_2)
- net GND: now also R3.1
- net Id+: now also R1.1

Commit message: Add Project Folder: KICAD
Parts:
- added RV1: 1K, Potentiometer_THT:Potentiometer_Bourns_3296W_Vertical, symbol Device:R_Potentiometer
- R2, R4: value 20k -> 100k
- R5: value 100 -> 150
Connections:
- net Out: now also RV1.2, RV1.3
- net at R2.2, R5.1, U1.1: now also RV1.1
Changed lines of the file:
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@@
+	)
+	(junction
+		(at 196.85 88.9)
+		(diameter 0)
+		(color 0 0 0 0)
 	)
 	(junction
@@
 	)
 	(junction
+		(at 196.85 95.25)
+		(diameter 0)
+		(color 0 0 0 0)
+	)
+	(junction
 		(at 104.14 99.06)
 		(diameter 0)
@@
 	)
 	(junction
-		(at 149.86 109.22)
+		(at 179.07 88.9)
 		(diameter 0)
 		(color 0 0 0 0)
@@
 	(wire
 		(pts
-			(xy 194.31 95.25) (xy 203.2 95.25)
+			(xy 194.31 95.25) (xy 196.85 95.25)
 		)
 		(stroke
@@
 	(wire
 		(pts
+			(xy 101.6 88.9) (xy 109.22 88.9)
+		)
+		(stroke
+			(width 0)
+			(type default)
+		)
+	)
+	(wire
+		(pts
 			(xy 157.48 82.55) (xy 162.56 82.55)
 		)
@@
 		)
 	)
+	(wire
+		(pts
+			(xy 196.85 85.09) (xy 196.85 88.9)
+		)
+		(stroke
+			(width 0)
+			(type default)
+		)
+	)
 	(polyline
 		(pts
@@
 	(wire
 		(pts
+			(xy 196.85 95.25) (xy 203.2 95.25)
+		)
+		(stroke
+			(width 0)
+			(type default)
+		)
+	)
+	(wire
+		(pts
 			(xy 203.2 95.25) (xy 203.2 106.68)
 		)
@@
 	(wire
 		(pts
-			(xy 149.86 109.22) (xy 149.86 118.11)
+			(xy 196.85 88.9) (xy 196.85 95.25)
 		)
 		(stroke
@@
 	(wire
 		(pts
+			(xy 179.07 88.9) (xy 179.07 95.25)
+		)
+		(stroke
+			(width 0)
+			(type default)
+		)
+	)
+	(wire
+		(pts
 			(xy 105.41 101.6) (xy 101.6 101.6)
 		)
@@
 	(wire
 		(pts
+			(xy 179.07 88.9) (xy 186.69 88.9)
+		)
+		(stroke
+			(width 0)
+			(type default)
+		)
+	)
+	(wire
+		(pts
 			(xy 162.56 82.55) (xy 162.56 92.71)
 		)
@@
 	(wire
 		(pts
+			(xy 190.5 85.09) (xy 196.85 85.09)
+		)
+		(stroke
+			(width 0)
+			(type default)
+		)
+	)
+	(wire
+		(pts
 			(xy 177.8 95.25) (xy 179.07 95.25)
 		)
@@
 		)
 	)
+	(wire
+		(pts
+			(xy 194.31 88.9) (xy 196.85 88.9)
+		)
+		(stroke
+			(width 0)
+			(type default)
+		)
+	)
 	(polyline
 		(pts
@@
 	(wire
 		(pts
-			(xy 139.7 91.44) (xy 139.7 90.17)
-		)
-		(stroke
-			(width 0)
-			(type default)
-		)
-	)
-	(wire
-		(pts
 			(xy 162.56 109.22) (xy 166.37 109.22)
 		)
@@
 	(wire
 		(pts
-			(xy 179.07 82.55) (xy 179.07 95.25)
+			(xy 179.07 82.55) (xy 179.07 88.9)
 		)
 		(stroke
@@
 			)
 		)
-		(property "Value" "20k"
+		(property "Value" "100k"
 			(at 170.18 82.55 90)
 			(show_name no)
@@
 	(symbol
 		(lib_id "power:GND")
-		(at 149.86 118.11 0)
+		(at 109.22 88.9 0)
+		(mirror y)
 		(unit 1)
 		(body_style 1)
@@
 		(in_pos_files yes)
 		(dnp no)
-		(fields_autoplaced yes)
 		(property "Reference" "#PWR08"
-			(at 149.86 124.46 0)
+			(at 109.22 95.25 0)
 			(hide yes)
 			(show_name no)
@@
 		)
 		(property "Value" "GND"
-			(at 149.86 123.19 0)
+			(at 109.22 93.98 0)
 			(show_name no)
 			(do_not_autoplace no)
@@
 		)
 		(property "Footprint" ""
-			(at 149.86 118.11 0)
+			(at 109.22 88.9 0)
 			(hide yes)
 			(show_name no)
@@
 		)
 		(property "Datasheet" ""
-			(at 149.86 118.11 0)
+			(at 109.22 88.9 0)
 			(hide yes)
 			(show_name no)
@@
 		)
 		(property "Description" "Power symbol creates a global label with name \"GND\" , ground"
-			(at 149.86 118.11 0)
+			(at 109.22 88.9 0)
 			(hide yes)
 			(show_name no)
@@
 	)
 	(symbol
+		(lib_id "Device:R_Potentiometer")
+		(at 190.5 88.9 90)
+		(unit 1)
+		(body_style 1)
+		(exclude_from_sim no)
+		(in_bom yes)
+		(on_board yes)
+		(in_pos_files yes)
+		(dnp no)
+		(property "Reference" "RV1"
+			(at 190.5 80.772 90)
+			(show_name no)
+			(do_not_autoplace no)
+			(effects
+				(font
+					(size 1.27 1.27)
+				)
+			)
+		)
+		(property "Value" "1K"
+			(at 190.5 83.312 90)
+			(show_name no)
+			(do_not_autoplace no)
+			(effects
+				(font
+					(size 1.27 1.27)
+				)
+			)
+		)
+		(property "Footprint" "Potentiometer_THT:Potentiometer_Bourns_3296W_Vertical"
+			(at 190.5 88.9 0)
+			(hide yes)
+			(show_name no)
+			(do_not_autoplace no)
+			(effects
+				(font
+					(size 1.27 1.27)
+				)
+			)
+		)
+		(property "Datasheet" ""
+			(at 190.5 88.9 0)
+			(hide yes)
+			(show_name no)
+			(do_not_autoplace no)
+			(effects
+				(font
+					(size 1.27 1.27)
+				)
+			)
+		)
+		(property "Description" "Potentiometer"
+			(at 190.5 88.9 0)
+			(hide yes)
+			(show_name no)
+			(do_not_autoplace no)
+			(effects
+				(font
+					(size 1.27 1.27)
+				)
+			)
+		)
+		(property "Sim.Device" "R"
+			(at 190.5 88.9 0)
+			(hide yes)
+			(show_name no)
+			(do_not_autoplace no)
+			(effects
+				(font
+					(size 1.27 1.27)
+				)
+			)
+		)
+		(property "Sim.Type" "POT"
+			(at 190.5 88.9 0)
+			(hide yes)
+			(show_name no)
+			(do_not_autoplace no)
+			(effects
+				(font
+					(size 1.27 1.27)
+				)
+			)
+		)
+		(property "Sim.Pins" "1=r0 2=wiper 3=r1"
+			(at 190.5 88.9 0)
+			(hide yes)
+			(show_name no)
+			(do_not_autoplace no)
+			(effects
+				(font
+					(size 1.27 1.27)
+				)
+			)
+		)
+		(pin "2"
+		)
+		(pin "3"
+		)
+		(pin "1"
+		)
+		(instances
+			(project "Howland-VCCS-TL072"
+				(path "/86a98f5b-8270-4f0f-bf90-6656280cb20e"
+					(reference "RV1")
+					(unit 1)
+				)
+			)
+		)
+	)
+	(symbol
 		(lib_id "Amplifier_Operational:TL072")
 		(at 78.74 95.25 0)
@@
 			)
 		)
-		(property "Value" "20k"
+		(property "Value" "100k"
 			(at 170.18 109.22 90)
 			(show_name no)
@@
 			)
 		)
-		(property "Value" "100"
+		(property "Value" "150"
 			(at 190.5 95.25 90)
 			(show_name no)
@@
 					(unit 1)
 				)
-			)
-		)
-	)
-	(symbol
-		(lib_id "power:GND")
-		(at 139.7 91.44 0)
-		(unit 1)
-		(body_style 1)
-		(exclude_from_sim no)
-		(in_bom yes)
-		(on_board yes)
-		(in_pos_files yes)
-		(dnp no)
-		(fields_autoplaced yes)
-		(property "Reference" "#PWR01"
-			(at 139.7 97.79 0)
-			(hide yes)
-			(show_name no)
-			(do_not_autoplace no)
-			(effects
-				(font
-					(size 1.27 1.27)
-				)
-			)
-		)
-		(property "Value" "GND"
-			(at 139.7 96.52 0)
-			(show_name no)
-			(do_not_autoplace no)
-			(effects
-				(font
-					(size 1.27 1.27)
-				)
-			)
-		)
-		(property "Footprint" ""
-			(at 139.7 91.44 0)
-			(hide yes)
-			(show_name no)
-			(do_not_autoplace no)
-			(effects
-				(font
-					(size 1.27 1.27)
-				)
-			)
-		)
-		(property "Datasheet" ""
-			(at 139.7 91.44 0)
-			(hide yes)
-			(show_name no)
-			(do_not_autoplace no)
-			(effects
-				(font
-					(size 1.27 1.27)
-				)
-			)
-		)
-		(property "Description" "Power symbol creates a global label with name \"GND\" , ground"
-			(at 139.7 91.44 0)
-			(hide yes)
-			(show_name no)
-			(do_not_autoplace no)
-			(effects
-				(font
-					(size 1.27 1.27)
-				)
-			)
-		)
-		(pin "1"
-		)
-		(instances
-			(project "Howland-VCCS-TL072"
-				(path "/86a98f5b-8270-4f0f-bf90-6656280cb20e"
-					(reference "#PWR01")
-					(unit 1)
-				)
