File: KiCAD/Howland-VCCS/Howland-VCCS-TL072-THT/Howland-VCCS-TL072-THT.kicad_pcb (KiCad board)
At the start: 2 copper layers, 43.2 x 25.4 mm, 9 parts, among them J1 Conn_01x03_Pin, J2 Conn_01x03_Pin, U1 TL072

Commit message: Add Project Folder: KICAD
Connections:
- J1 pad 2: GND -> /Id-
- R3 pad 1: GND -> /Id-
Routing:
- net /Id-: track 0.00 -> 42.3 mm
- net GND: track 40.8 -> 0.00 mm
Other:
- board text added: "GND"
- board text added: "IN+"
- board text added: "IN-"
- board text added: "OUT"
- board text added: "VCC"
- board text added: "VEE"

Commit message: Add Project Folder: KICAD
Other:
- board text added: "Discrete VCCS - TL072 Ver.1.2 20-10-26"

Commit message: Add Project Folder: KICAD
Parts:
- added G***: LOGO, LOGO, B.Cu at (162.0, 96.6)

Commit message: Add Project Folder: KICAD
Parts:
- removed G***: LOGO, LOGO
