File: KiCAD/ATMega16-STM32 BP Adapter/ATMega16-STM32 BP Adapter_THT/ATMega16-STM32 BP Adapter_THT.kicad_sch (KiCad schematic)
At the start: 0 parts

Commit message: Add Project Folder: KICAD
Parts:
- added J1, J2: Conn_01x20, symbol Connector_Generic:Conn_01x20
- added U2: YAAJ_BluePill_Part_Like, symbol MCU:YAAJ_BluePill_Part_Like

Commit message: Add Project Folder: KICAD
Parts:
- added J3, J4: Conn_01x20, Connector_PinHeader_2.54mm:PinHeader_1x20_P2.54mm_Vertical, symbol Connector_Generic:Conn_01x20
- J1, J2: footprint (none) -> Connector_PinSocket_2.54mm:PinSocket_1x20_P2.54mm_Vertical
- U2: footprint (none) -> MCU_Custom:BLUEPILL_SILKSCREEN
Connections:
- net GND: now also J1.1 (Pin_1), J1.2 (Pin_2), J2.19 (Pin_19), U2.19 (GND), U2.39 (GND), U2.40 (GND), J3.10 (Pin_10), J4.11 (Pin_11)
- net VCC: now also J4.10 (Pin_10)
- net ATM16.PB4: now reaches J2.1 (Pin_1)
- net ATM16.PB4: now also U2.1 (PB12), J4.5 (Pin_5)
- net ATM16.PB3: now reaches J2.11 (Pin_11)
- net ATM16.PB3: now also U2.11 (PB3), J4.4 (Pin_4)
- net ATM16.PD7: now reaches J2.12 (Pin_12)
- net ATM16.PD7: now also U2.12 (PB4), J3.20 (Pin_20)
- net ATM16.PC0: now reaches J2.14 (Pin_14)
- net ATM16.PC0: now also U2.14 (PB6), J3.19 (Pin_19)
- net ATM16.PC1: now reaches J2.15 (Pin_15)
- net ATM16.PC1: now also U2.15 (PB7), J3.18 (Pin_18)
- net ATM16.PD2: now reaches J2.16 (Pin_16)
- net ATM16.PD2: now also U2.16 (PB8), J4.16 (Pin_16)
- net ATM16.PD3: now reaches J2.17 (Pin_17)
- net ATM16.PD3: now also U2.17 (PB9), J4.17 (Pin_17)
- net 5V: now reaches J2.18 (Pin_18)
- net 5V: now also U2.18 (5V)
- net ATM16.PB7: now reaches J2.2 (Pin_2)
- net ATM16.PB7: now also U2.2 (PB13), J4.8 (Pin_8)
- net 3V3: now reaches J2.20 (Pin_20)
- net 3V3: now also J1.3 (Pin_3), U2.20 (3V3), U2.38 (3V3)
- net ATM16.PB6: now reaches J2.3 (Pin_3)
- net ATM16.PB6: now also U2.3 (PB14), J4.7 (Pin_7)
- net ATM16.PB5: now reaches J2.4 (Pin_4)
- net ATM16.PB5: now also U2.4 (PB15), J4.6 (Pin_6)
- net ATM16.PD4: now reaches J2.5 (Pin_5)
- net ATM16.PD4: now also U2.5 (PA8), J4.18 (Pin_18)
- net ATM16.PD1: now reaches J2.6 (Pin_6)
- net ATM16.PD1: now also U2.6 (PA9), J4.15 (Pin_15)
- net ATM16.PD0: now reaches J2.7 (Pin_7)
- net ATM16.PD0: now also U2.7 (PA10), J4.14 (Pin_14)
- net ATM16.PB1: now reaches J2.9 (Pin_9)
- net ATM16.PB1: now also U2.9 (PA12), J4.2 (Pin_2)
- net ADC6: now reaches J1.10 (Pin_10)
- net ADC6: now also U2.31 (PA6), J3.7 (Pin_7)
- net ADC5: now reaches J1.11 (Pin_11)
- net ADC5: now also U2.30 (PA5), J3.6 (Pin_6)
- net ADC4: now reaches J1.12 (Pin_12)
- net ADC4: now also U2.29 (PA4), J3.5 (Pin_5)
- net ADC3: now reaches J1.13 (Pin_13)
- net ADC3: now also U2.28 (PA3), J3.4 (Pin_4)
- net ADC2: now reaches J1.14 (Pin_14)
- net ADC2: now also U2.27 (PA2), J3.3 (Pin_3)
- net ADC1: now reaches J1.15 (Pin_15)
- net ADC1: now also U2.26 (PA1), J3.2 (Pin_2)
- net ADC0: now reaches J1.16 (Pin_16)
- net ADC0: now also U2.25 (PA0), J3.1 (Pin_1)
- net ATM16.PC7: now reaches J1.17 (Pin_17)
- net ATM16.PC7: now also U2.24 (PC15), J3.12 (Pin_12)
- net ATM16.PC6: now reaches J1.18 (Pin_18)
- net ATM16.PC6: now also U2.23 (PC14), J3.13 (Pin_13)
- net ATM16.RESET: now reaches J1.4 (Pin_4)
- net ATM16.RESET: now also U2.37 (RST), J4.9 (Pin_9)
- net ATM16.PB0: now reaches J1.6 (Pin_6)
- net ATM16.PB0: now also U2.35 (PB10), J4.1 (Pin_1)
- net ATM16.PD6: now reaches J1.7 (Pin_7)
- net ATM16.PD6: now also U2.34 (PB1), J4.20 (Pin_20)
- net ATM16.PD5: now reaches J1.8 (Pin_8)
- net ATM16.PD5: now also U2.33 (PB0), J4.19 (Pin_19)
- net ADC7: now reaches J1.9 (Pin_9)
- net ADC7: now also U2.32 (PA7), J3.8 (Pin_8)
- new net ATM16.PB2: J4.3 (Pin_3)
- new net ATM16.PC2: J3.17 (Pin_17)
- new net ATM16.PC3: J3.16 (Pin_16)
- new net ATM16.PC4: J3.15 (Pin_15)
- new net ATM16.PC5: J3.14 (Pin_14)
- no-connect marks 0 -> 16
Other:
- moved on the sheet: J1, J2, U2
